Commit message: cleaning up

File: teambowl_ws/src/bringup/robot_description/bowl.urdf (robot description, URDF)
Before this commit: robot bowl, 21 links, 20 joints
Links:
- link Align bar: geometry visual mesh filename=package://bringup/robot_description/meshes/83.stl scale=1 1 1
- link Align bar_1: geometry visual mesh filename=package://bringup/robot_description/meshes/83.stl scale=1 1 1
- link Calf: geometry visual mesh filename=package://bringup/robot_description/meshes/113.stl scale=1 1 1
- link Calf_1: geometry visual mesh filename=package://bringup/robot_description/meshes/113.stl scale=1 1 1
- link Foot: geometry visual mesh filename=package://bringup/robot_description/meshes/109.stl scale=1 1 1
- link Foot_1: geometry visual mesh filename=package://bringup/robot_description/meshes/109.stl scale=1 1 1
- link Frame: geometry visual mesh filename=package://bringup/robot_description/meshes/102.stl scale=1 1 1
- link Hip: geometry visual mesh filename=package://bringup/robot_description/meshes/59.stl scale=1 1 1
- link Hip_1: geometry visual mesh filename=package://bringup/robot_description/meshes/59.stl scale=1 1 1
- link Knee Kicker: geometry visual mesh filename=package://bringup/robot_description/meshes/87.stl scale=1 1 1
- link Knee Kicker_1: geometry visual mesh filename=package://bringup/robot_description/meshes/87.stl scale=1 1 1
- link Lid: geometry visual mesh filename=package://bringup/robot_description/meshes/95.stl scale=1 1 1
- link Lid Gear: geometry visual mesh filename=package://bringup/robot_description/meshes/63.stl scale=1 1 1
- link Thigh: geometry visual mesh filename=package://bringup/robot_description/meshes/79.stl scale=1 1 1
- link Thigh_1: geometry visual mesh filename=package://bringup/robot_description/meshes/79.stl scale=1 1 1
- link Wheel: geometry visual mesh filename=package://bringup/robot_description/meshes/132.stl scale=1 1 1
- link Wheel Gear: geometry visual mesh filename=package://bringup/robot_description/meshes/91.stl scale=1 1 1
- link Wheel Gear_1: geometry visual mesh filename=package://bringup/robot_description/meshes/91.stl scale=1 1 1
- link Wheel_1: geometry visual mesh filename=package://bringup/robot_description/meshes/132.stl scale=1 1 1
- link z_axis: geometry visual mesh filename=package://bringup/robot_description/meshes/75.stl scale=1 1 1

Commit message: new URDF and more cleanup

File: teambowl_ws/src/bringup/robot_description/bowl.urdf (robot description, URDF)
Before this commit: robot bowl, 21 links, 20 joints
Links:
- added link z_axis_1, mass 4.90874e-07; visual mesh filename=package://bowl/meshes/75.stl scale=1 1 1
- added link z_axis_2, mass 4.90874e-07; visual mesh filename=package://bowl/meshes/75.stl scale=1 1 1
- added link z_axis_3, mass 4.90874e-07; visual mesh filename=package://bowl/meshes/75.stl scale=1 1 1
- link Align bar: geometry visual mesh filename=package://bowl/meshes/83.stl scale=1 1 1
- link Align bar_1: geometry visual mesh filename=package://bowl/meshes/83.stl scale=1 1 1
- link Calf: geometry visual mesh filename=package://bowl/meshes/131.stl scale=1 1 1
- link Calf_1: geometry visual mesh filename=package://bowl/meshes/131.stl scale=1 1 1
- link Foot: geometry visual mesh filename=package://bowl/meshes/127.stl scale=1 1 1
- link Foot_1: geometry visual mesh filename=package://bowl/meshes/127.stl scale=1 1 1
- link Frame: mass 0.00445655 -> 0.00493951; geometry visual mesh filename=package://bowl/meshes/111.stl scale=1 1 1
- link Hip: geometry visual mesh filename=package://bowl/meshes/59.stl scale=1 1 1
- link Hip_1: geometry visual mesh filename=package://bowl/meshes/59.stl scale=1 1 1
- link Knee Kicker: geometry visual mesh filename=package://bowl/meshes/87.stl scale=1 1 1
- link Knee Kicker_1: geometry visual mesh filename=package://bowl/meshes/87.stl scale=1 1 1
- link Lid: mass 0.00148516 -> 0.00166483; geometry visual mesh filename=package://bowl/meshes/104.stl scale=1 1 1
- link Lid Gear: geometry visual mesh filename=package://bowl/meshes/63.stl scale=1 1 1
- link Thigh: geometry visual mesh filename=package://bowl/meshes/79.stl scale=1 1 1
- link Thigh_1: geometry visual mesh filename=package://bowl/meshes/79.stl scale=1 1 1
- link Wheel: geometry visual mesh filename=package://bowl/meshes/150.stl scale=1 1 1
- link Wheel Gear: geometry visual mesh filename=package://bowl/meshes/100.stl scale=1 1 1
- link Wheel Gear_1: geometry visual mesh filename=package://bowl/meshes/100.stl scale=1 1 1
- link Wheel_1: geometry visual mesh filename=package://bowl/meshes/150.stl scale=1 1 1
- link z_axis: geometry visual mesh filename=package://bowl/meshes/75.stl scale=1 1 1
Joints:
- removed joint closing_knee0_0
- removed joint dof_ankle0_0
- removed joint dof_calf0_0
- removed joint dof_driver0_0
- removed joint dof_hip0_0
- removed joint dof_lid_0
- removed joint dof_lid_gear_0
- removed joint dof_motor0_0
- removed joint dof_motor1_0
- removed joint dof_trochanter0_0
- added joint ankle0_0: type continuous, parent Calf_1, child Foot_1, origin xyz=0.02725 0.0957158 -0.279381 rpy=0.610865 -2.01631e-15 -1.5672e-15, axis -1 -1.69007e-15 -1.55165e-15
- added joint calf0_0: type continuous, parent Hip_1, child Thigh_1, origin xyz=-0.03125 -0.07 -3.19189e-15 rpy=-0.436332 5.52108e-15 -5.14189e-17, axis -1 -2.87471e-15 -1.34042e-16
- added joint driver0_0: type continuous, parent Hip_1, child Knee Kicker, origin xyz=0.03125 -0.07 3.78864e-15 rpy=-0.785398 -3.16395e-15 1.06414e-15, axis 1 2.42762e-15 1.53802e-17
- added joint hip0_0: type continuous, parent Frame, child Hip_1, origin xyz=-0.155463 -0.03389 -0.118135 rpy=-6.79796e-15 -1.13089e-14 -4.9225e-14, axis 3.88364e-16 1 -2.60209e-17
- added joint knee0_0: type continuous, parent Thigh_1, child Calf_1, origin xyz=0.02625 -0.225522 0.190669 rpy=-0.349066 8.47614e-15 -3.25427e-15, axis 1 2.68293e-15 3.68387e-17
- added joint left_mono_0: type fixed, parent Frame, child z_axis_3, origin xyz=-0.0429629 0.229702 0.0818872 rpy=-1.5708 -5.51779e-30 -6.56158e-18, axis 0 0 -1
- added joint left_motor_0: type continuous, parent Frame, child Wheel Gear_1, origin xyz=-0.282193 0.0390428 0.0543905 rpy=-1.5708 7.96232e-17 7.96232e-17, axis 1 -7.94831e-31 -7.96232e-17
- added joint lid_0: type continuous, parent Frame, child Lid, origin xyz=-0.00546297 -0.11133 0.294511 rpy=1.69673e-18 1.50366e-19 -3.13011e-36, axis -1.50366e-19 2.25134e-17 1
- added joint lid_gear_0: type continuous, parent Frame, child Lid Gear, origin xyz=-0.00560326 -0.163819 0.240861 rpy=-7.24987e-17 -2.11965e-17 4.41241e-34, axis -2.11965e-17 5.1682e-17 -1
- added joint rgb_cam_0: type fixed, parent Frame, child z_axis_1, origin xyz=-0.00546292 0.229702 0.0818872 rpy=-1.5708 -5.51779e-30 -6.56158e-18, axis 0 0 -1
- added joint right_mono_0: type fixed, parent Frame, child z_axis_2, origin xyz=0.0320371 0.229702 0.0818872 rpy=-1.5708 -5.51779e-30 -6.56158e-18, axis 0 0 -1
- added joint right_motor_0: type continuous, parent Frame, child Wheel Gear, origin xyz=0.271267 0.0390428 0.0543905 rpy=5.78468e-34 -1.7632e-16 -6.56158e-18, axis 1 -7.94831e-31 -7.96232e-17
- added joint trochanter0_0: type continuous, parent Knee Kicker, child Align bar_1, origin xyz=-0.03625 -0.0225108 0.0657059 rpy=0.349066 3.83054e-15 1.27368e-15, axis -1 -2.3946e-15 -1.19973e-16
- joint closing_knee1_0: origin xyz=0.02625 -0.225522 0.190669 rpy=-0.349066 1.37701e-15 9.32681e-16 -> xyz=0.02625 -0.225522 0.190669 rpy=-0.349066 -7.96611e-16 -1.31473e-14
- joint dof_ankle1_0: origin xyz=0.02725 0.0957158 -0.279381 rpy=0.610865 1.67124e-15 1.43103e-15 -> xyz=0.02725 0.0957158 -0.279381 rpy=0.610865 1.67033e-15 1.4304e-15
- joint dof_calf1_0: origin xyz=-0.03125 -0.07 3.23352e-15 rpy=-0.436332 -1.23267e-15 -1.29098e-14 -> xyz=-0.03125 -0.07 3.21965e-15 rpy=-0.436332 6.36257e-15 -1.23128e-14
- joint dof_driver1_0: origin xyz=0.03125 -0.07 1.01308e-14 rpy=-0.785398 3.02832e-16 -1.26566e-14 -> xyz=0.03125 -0.07 1.02696e-14 rpy=-0.785398 3.02832e-16 -1.93215e-15
- joint dof_hip1_0: origin xyz=0.144537 -0.03389 -0.118135 rpy=3.18538e-16 -1.87654e-15 3.19124e-14 -> xyz=0.144537 -0.03389 -0.118135 rpy=-6.76723e-15 -1.26908e-14 -4.91142e-14
- joint left_wheel_0: axis 1 6.56158e-18 8.86235e-18 -> -1 -6.56158e-18 -8.86235e-18; origin xyz=-0.302263 -0.03839 -0.056195 rpy=-0.110825 6.43831e-18 -1.48663e-17 -> xyz=-0.302263 -0.03839 -0.056195 rpy=1.73472e-17 -8.50584e-19 4.81092e-17
- joint right_wheel_0: origin xyz=0.26638 -0.03839 -0.056195 rpy=-3.14159 -1.30343e-17 -3.14159 -> xyz=0.26638 -0.03839 -0.056195 rpy=3.14159 -1.30343e-17 -3.14159
